File: pcb_smartlock.kicad_sch (KiCad schematic)
At the start: 61 parts, among them IC1 ST25R3918-AQET, J1 Conn_01x02, J2 Conn_01x03, Q3 IRLML6344TRPBF, Q4 IRLML6344TRPBF, SW1 SKSCLBE010, SW2 SKSCLBE010, SW3 SKSCLBE010, U2 SPX3819M5-L-1-8, U3 ESP32-C3-MINI-1-H4X, U5 SPX3819M5-L-1-8

Commit message: Add silkscreen
Parts:
- C10: value 10uf -> 10uF
- C11, C19: value 1uf -> 1uF
- C12: value 10u -> 10uF
- C13: value 100n -> 0.1uF
- C15, C20: value 2.2u -> 2.2uF
- C7, C8, C9: value 0.1u -> 0.1uF
- R4: value 5.1K -> 5.1k

Commit message: add Interactive BOM HTML
Parts:
- C9: footprint Capacitor_SMD:C_0603_1608Metric_Pad1.08x0.95mm_HandSolder -> Capacitor_SMD:C_0603_1608Metric_Pad1.08x0.95mm
- SP1: value ~ -> (none)

Commit message: Edit MOSFET & Schottky to pick available ones
Parts:
- D4, D5: value b5819WS -> SBA130CH-AU_R1_000A1; footprint Diode_SMD:D_0603_1608Metric -> SBA130CH-AU_R1_000A1:SOD-323HE
Changed lines of the file:
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@@
 			)
 		)
-		(property "Value" "b5819WS"
-			(at 260.604 151.384 0)
-			(show_name no)
-			(do_not_autoplace no)
-			(effects
-				(font
-					(size 1.27 1.27)
-				)
-			)
-		)
-		(property "Footprint" "Diode_SMD:D_0603_1608Metric"
+		(property "Value" "SBA130CH-AU_R1_000A1"
+			(at 259.334 151.13 0)
+			(show_name no)
+			(do_not_autoplace no)
+			(effects
+				(font
+					(size 1.27 1.27)
+				)
+			)
+		)
+		(property "Footprint" "SBA130CH-AU_R1_000A1:SOD-323HE"
 			(at 260.35 148.59 0)
 			(hide yes)
@@
 			)
 		)
-		(property "Datasheet" ""
+		(property "Datasheet" "https://www.mouser.fr/datasheet/3/3736/1/11145663EF9055F8C188C22CC003165FC5A818A8439A953D3A6E1D8FCBF51DA1.pdf"
 			(at 260.35 148.59 0)
 			(hide yes)
@@
 			)
 		)
-		(property "Value" "b5819WS"
-			(at 103.124 80.264 0)
-			(show_name no)
-			(do_not_autoplace no)
-			(effects
-				(font
-					(size 1.27 1.27)
-				)
-			)
-		)
-		(property "Footprint" "Diode_SMD:D_0603_1608Metric"
+		(property "Value" "SBA130CH-AU_R1_000A1"
+			(at 102.87 90.678 0)
+			(show_name no)
+			(do_not_autoplace no)
+			(effects
+				(font
+					(size 1.27 1.27)
+				)
+			)
+		)
+		(property "Footprint" "SBA130CH-AU_R1_000A1:SOD-323HE"
 			(at 102.87 77.47 0)
 			(hide yes)
@@
 			)
 		)
-		(property "Datasheet" ""
+		(property "Datasheet" "https://www.mouser.fr/datasheet/3/3736/1/11145663EF9055F8C188C22CC003165FC5A818A8439A953D3A6E1D8FCBF51DA1.pdf"
 			(at 102.87 77.47 0)
 			(hide yes)
